File: Project_Roll.kicad_pcb (KiCad board)
At the start: 4 copper layers, 98.2 x 122 mm, 75 parts, among them J1 TB002-500-02BE, J10 Conn_01x04, J11 Conn_01x04, J12 Conn_01x02, J13 TB002-500-02BE, J14 TB002-500-02BE, J15 TB002-500-02BE, J16 TB002-500-02BE, J17 Conn_01x03, J2 TB002-500-02BE, J3 TB002-500-02BE, J4 TB002-500-02BE, J5 TB002-500-02BE, J6 Conn_01x05, J7 Conn_01x05, J8 Conn_01x04, J9 Conn_01x04, Q1 IRFS7430TRLPBF, U1 AP62300TWU, U2 GY-521, U3 ESP32-DEVKIT-V1, U4 MIC5504-3.3YM5

Commit message: Separated schematic into sheets
Routing:
- net GND: vias 199 -> 256
- added copper zone on B.Cu, net Net-(D3-A1)
